File: KiCad/ScoreController/ScoreController/ScoreController.kicad_pcb (KiCad board)
At the start: 2 copper layers, 70.3 x 60 mm, 23 parts, among them J1 Conn_01x02, J10 Conn_01x03, J11 Conn_01x02, J12 Conn_01x03, J13 Conn_01x02, J14 Conn_01x03, J15 Conn_01x02, J2 Conn_01x02, J3 Conn_01x03, J4 Conn_01x11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

Commit message: Something broke in the previous 2 commits beforore this one
Parts:
- J6: footprint TerminalBlock_4Ucon:TerminalBlock_4Ucon_1x02_P3.50mm_Horizontal -> Connector_JST:JST_XH_B2B-XH-A_1x02_P2.50mm_Vertical
- U1: footprint Pi-Pico:RPi_Pico_SMD -> RPi_Pico:RPi_Pico_SMD_TH
- moved J6 2.90 mm to (156.9, 62.3), turned to 0 degrees
Routing:
- net /3V3: track 186.6 -> 207.4 mm, vias 3 -> 5
- net /DISPLAY_SCK: track 17.0 -> 19.8 mm, vias 1 -> 2
- net /GND: track 17.5 -> 19.7 mm
- net /DISPLAY_MOSI: track 12.5 -> 11.8 mm
- net /5V: track 0.50 -> 0.00 mm
Other:
- board text added: "Score Controller Designed by Mark Hutcheson March 2022 updated Nov 2022"
- board text removed: "Score Controller Designed by Mark Hutcheson March 2022"
